Commit message: update the limits

File: Hand/Hand_left/URDF_L.urdf (robot description, URDF)
Before this commit: robot URDF_0605_L, 24 links, 23 joints
Joints:
- joint F1-L-DIP: limit lower=-0.35 upper=1.31 effort=1.7 velocity=4.88 -> lower=-0.4363323 upper=1.3962634 effort=1.7 velocity=4.88
- joint F1-L-MCP1: limit lower=-0.52 upper=0.785 effort=6.0 velocity=3.84 -> lower=-0.6108652 upper=0.8726646 effort=6.0 velocity=3.84
- joint F1-L-MCP2: limit lower=-0.35 upper=0.61 effort=6.5 velocity=2.82 -> lower=-0.4363323 upper=0.7853982 effort=6.5 velocity=2.82
- joint F1-L-PIP: limit lower=-0.35 upper=1.31 effort=3.5 velocity=4.88 -> lower=-0.5235988 upper=1.3089969 effort=3.5 velocity=4.88
- joint F2-L-DIP: limit lower=0 upper=1.22 effort=1.5 velocity=3.59 -> lower=-0.0872665 upper=1.3089969 effort=1.5 velocity=3.59
- joint F2-L-MCP1: limit lower=-0.52 upper=1.57 effort=5.5 velocity=6.15 -> lower=-0.6108652 upper=1.6580628 effort=5.5 velocity=6.15
- joint F2-L-MCP2: limit lower=-0.61 upper=0.61 effort=6.0 velocity=3.59 -> lower=-0.6981317 upper=0.6981317 effort=6.0 velocity=3.59; origin xyz=0.04512 0.078019 0.00395 rpy=3.1416 0 3.1416 -> xyz=0.04512 0.078019 0.00395 rpy=3.1416 0 2.8798
- joint F2-L-PIP: limit lower=0 upper=1.92 effort=3.0 velocity=5.65 -> lower=-0.0872665 upper=1.8325957 effort=3.0 velocity=5.65
- joint F3-L-DIP: limit lower=0 upper=1.22 effort=1.5 velocity=3.59 -> lower=-0.0872665 upper=1.3089969 effort=1.5 velocity=3.59
- joint F3-L-MCP1: limit lower=-0.52 upper=1.57 effort=5.5 velocity=6.15 -> lower=-0.6108652 upper=1.6580628 effort=5.5 velocity=6.15
- joint F3-L-MCP2: limit lower=-0.61 upper=0.61 effort=6.0 velocity=3.59 -> lower=-0.6981317 upper=0.6108652 effort=6.0 velocity=3.59
- joint F3-L-PIP: limit lower=0 upper=1.92 effort=3.0 velocity=5.65 -> lower=-0.0872665 upper=1.8325957 effort=3.0 velocity=5.65
- joint F4-L-DIP: limit lower=0 upper=1.22 effort=1.5 velocity=3.59 -> lower=-0.0872665 upper=1.3089969 effort=1.5 velocity=3.59
- joint F4-L-MCP1: limit lower=-0.52 upper=1.57 effort=5.5 velocity=6.15 -> lower=-0.6108652 upper=1.6580628 effort=5.5 velocity=6.15
- joint F4-L-MCP2: limit lower=-0.61 upper=0.61 effort=6.0 velocity=3.59 -> lower=-0.6981317 upper=0.5235988 effort=6.0 velocity=3.59; origin xyz=0.0059875 0.078019 0.00395 rpy=3.1416 0 3.1416 -> xyz=0.0059875 0.078019 0.00395 rpy=3.1416 0 3.4034
- joint F4-L-PIP: limit lower=0 upper=1.92 effort=3.0 velocity=5.65 -> lower=-0.0872665 upper=1.8325957 effort=3.0 velocity=5.65
- joint F5-L-DIP: limit lower=0 upper=1.22 effort=1.5 velocity=3.59 -> lower=-0.0872665 upper=1.3089969 effort=1.5 velocity=3.59
- joint F5-L-MCP1: limit lower=-0.52 upper=1.57 effort=5.5 velocity=6.15 -> lower=-0.6108652 upper=1.6580628 effort=5.5 velocity=6.15
- joint F5-L-MCP2: limit lower=-0.61 upper=0.61 effort=6.0 velocity=3.59 -> lower=-0.6981317 upper=0.6981317 effort=6.0 velocity=3.59; origin xyz=-0.01361 0.063366 0.00395 rpy=3.1416 0 3.1416 -> xyz=-0.01361 0.063366 0.00395 rpy=3.1416 0 3.7350
- joint F5-L-PIP: limit lower=0 upper=1.92 effort=3.0 velocity=5.65 -> lower=-0.0872665 upper=1.8325957 effort=3.0 velocity=5.65
- joint PALM-L: limit lower=-1.22 upper=1.22 effort=10.0 velocity=2.5 -> lower=-0.7853982 upper=0.7853982 effort=10.0 velocity=2.5
- joint WRIST-PALM-L: limit lower=-0.785 upper=0.785 effort=12.0 velocity=2.0 -> lower=-1.2217305 upper=1.2217305 effort=12.0 velocity=2.0

File: Hand/Hand_right/URDF_R.urdf (robot description, URDF)
Before this commit: robot URDF_0605_R, 24 links, 23 joints
Joints:
- joint F1-R-DIP: limit lower=-0.35 upper=1.31 effort=1.7 velocity=4.88 -> lower=-0.4363323 upper=1.3962634 effort=1.7 velocity=4.88
- joint F1-R-MCP1: limit lower=-0.52 upper=0.785 effort=6.0 velocity=3.84 -> lower=-0.6108652 upper=0.8726646 effort=6.0 velocity=3.84
- joint F1-R-MCP2: limit lower=-0.35 upper=0.61 effort=6.5 velocity=2.82 -> lower=-0.4363323 upper=0.7853982 effort=6.5 velocity=2.82
- joint F1-R-PIP: limit lower=-0.35 upper=1.31 effort=3.5 velocity=4.88 -> lower=-0.5235988 upper=1.3089969 effort=3.5 velocity=4.88
- joint F2-R-DIP: limit lower=0 upper=1.22 effort=1.5 velocity=3.59 -> lower=-0.0872665 upper=1.3089969 effort=1.5 velocity=3.59
- joint F2-R-MCP1: limit lower=-0.52 upper=1.57 effort=5.5 velocity=6.15 -> lower=-0.6108652 upper=1.6580628 effort=5.5 velocity=6.15
- joint F2-R-MCP2: limit lower=-0.61 upper=0.61 effort=6.0 velocity=3.59 -> lower=-0.6981317 upper=0.6981317 effort=6.0 velocity=3.59; origin xyz=0.0475313 0.0778613 0.0023 rpy=0 0 0 -> xyz=0.0475313 0.0778613 0.0023 rpy=0 0 -0.2618
- joint F2-R-PIP: limit lower=0 upper=1.92 effort=3.0 velocity=5.65 -> lower=-0.0872665 upper=1.8325957 effort=3.0 velocity=5.65
- joint F3-R-DIP: limit lower=0 upper=1.22 effort=1.5 velocity=3.59 -> lower=-0.0872665 upper=1.3089969 effort=1.5 velocity=3.59
- joint F3-R-MCP1: limit lower=-0.52 upper=1.57 effort=5.5 velocity=6.15 -> lower=-0.6108652 upper=1.6580628 effort=5.5 velocity=6.15
- joint F3-R-MCP2: limit lower=-0.61 upper=0.61 effort=6.0 velocity=3.59 -> lower=-0.6981317 upper=0.6108652 effort=6.0 velocity=3.59
- joint F3-R-PIP: limit lower=0 upper=1.92 effort=3.0 velocity=5.65 -> lower=-0.0872665 upper=1.8325957 effort=3.0 velocity=5.65
- joint F4-R-DIP: limit lower=0 upper=1.22 effort=1.5 velocity=3.59 -> lower=-0.0872665 upper=1.3089969 effort=1.5 velocity=3.59
- joint F4-R-MCP1: limit lower=-0.52 upper=1.57 effort=5.5 velocity=6.15 -> lower=-0.6108652 upper=1.6580628 effort=5.5 velocity=6.15
- joint F4-R-MCP2: limit lower=-0.61 upper=0.61 effort=6.0 velocity=3.59 -> lower=-0.6981317 upper=0.5235988 effort=6.0 velocity=3.59; origin xyz=0.008399 0.0778613 0.0023 rpy=0 0 0 -> xyz=0.008399 0.0778613 0.0023 rpy=0 0 0.2618
- joint F4-R-PIP: limit lower=0 upper=1.92 effort=3.0 velocity=5.65 -> lower=-0.0872665 upper=1.8325957 effort=3.0 velocity=5.65
- joint F5-R-DIP: limit lower=0 upper=1.22 effort=1.5 velocity=3.59 -> lower=-0.0872665 upper=1.3089969 effort=1.5 velocity=3.59
- joint F5-R-MCP1: limit lower=-0.52 upper=1.57 effort=5.5 velocity=6.15 -> lower=-0.6108652 upper=1.6580628 effort=5.5 velocity=6.15
- joint F5-R-MCP2: limit lower=-0.61 upper=0.61 effort=6.0 velocity=3.59 -> lower=-0.6981317 upper=0.6981317 effort=6.0 velocity=3.59; origin xyz=-0.0111988 0.0632092 0.0023 rpy=0 0 0 -> xyz=-0.0111988 0.0632092 0.0023 rpy=0 0 0.5934
- joint F5-R-PIP: limit lower=0 upper=1.92 effort=3.0 velocity=5.65 -> lower=-0.0872665 upper=1.8325957 effort=3.0 velocity=5.65
- joint PALM-R: limit lower=-1.22 upper=1.22 effort=10.0 velocity=2.5 -> lower=-0.7853982 upper=0.7853982 effort=10.0 velocity=2.5
- joint WRIST-PALM-R: limit lower=-0.785 upper=0.785 effort=12.0 velocity=2.0 -> lower=-1.2217305 upper=1.2217305 effort=12.0 velocity=2.0

File: bimanualHand/openarm_hand_bimanual.urdf (robot description, URDF)
Before this commit: robot openarm_hand_bimanual, 62 links, 61 joints
Joints:
- joint F1-L-DIP: limit lower=-0.35 upper=1.31 effort=1.7 velocity=4.88 -> lower=-0.4363323 upper=1.3962634 effort=1.7 velocity=4.88
- joint F1-L-MCP1: limit lower=-0.52 upper=0.785 effort=6.0 velocity=3.84 -> lower=-0.6108652 upper=0.8726646 effort=6.0 velocity=3.84
- joint F1-L-MCP2: limit lower=-0.35 upper=0.61 effort=6.5 velocity=2.82 -> lower=-0.4363323 upper=0.7853982 effort=6.5 velocity=2.82
- joint F1-L-PIP: limit lower=-0.35 upper=1.31 effort=3.5 velocity=4.88 -> lower=-0.5235988 upper=1.3089969 effort=3.5 velocity=4.88
- joint F1-R-DIP: limit lower=-0.35 upper=1.31 effort=1.7 velocity=4.88 -> lower=-0.4363323 upper=1.3962634 effort=1.7 velocity=4.88
- joint F1-R-MCP1: limit lower=-0.52 upper=0.785 effort=6.0 velocity=3.84 -> lower=-0.6108652 upper=0.8726646 effort=6.0 velocity=3.84
- joint F1-R-MCP2: limit lower=-0.35 upper=0.61 effort=6.5 velocity=2.82 -> lower=-0.4363323 upper=0.7853982 effort=6.5 velocity=2.82
- joint F1-R-PIP: limit lower=-0.35 upper=1.31 effort=3.5 velocity=4.88 -> lower=-0.5235988 upper=1.3089969 effort=3.5 velocity=4.88
- joint F2-L-DIP: limit lower=0 upper=1.22 effort=1.5 velocity=3.59 -> lower=-0.0872665 upper=1.3089969 effort=1.5 velocity=3.59
- joint F2-L-MCP1: limit lower=-0.52 upper=1.57 effort=5.5 velocity=6.15 -> lower=-0.6108652 upper=1.6580628 effort=5.5 velocity=6.15
- joint F2-L-MCP2: limit lower=-0.61 upper=0.61 effort=6.0 velocity=3.59 -> lower=-0.6981317 upper=0.6981317 effort=6.0 velocity=3.59; origin xyz=0.04512 0.078019 0.00395 rpy=3.1416 0 3.1416 -> xyz=0.04512 0.078019 0.00395 rpy=3.1416 0 2.8798
- joint F2-L-PIP: limit lower=0 upper=1.92 effort=3.0 velocity=5.65 -> lower=-0.0872665 upper=1.8325957 effort=3.0 velocity=5.65
- joint F2-R-DIP: limit lower=0 upper=1.22 effort=1.5 velocity=3.59 -> lower=-0.0872665 upper=1.3089969 effort=1.5 velocity=3.59
- joint F2-R-MCP1: limit lower=-0.52 upper=1.57 effort=5.5 velocity=6.15 -> lower=-0.6108652 upper=1.6580628 effort=5.5 velocity=6.15
- joint F2-R-MCP2: limit lower=-0.61 upper=0.61 effort=6.0 velocity=3.59 -> lower=-0.6981317 upper=0.6981317 effort=6.0 velocity=3.59; origin xyz=0.0475313 0.0778613 0.0023 rpy=0 0 0 -> xyz=0.0475313 0.0778613 0.0023 rpy=0 0 -0.2618
- joint F2-R-PIP: limit lower=0 upper=1.92 effort=3.0 velocity=5.65 -> lower=-0.0872665 upper=1.8325957 effort=3.0 velocity=5.65
- joint F3-L-DIP: limit lower=0 upper=1.22 effort=1.5 velocity=3.59 -> lower=-0.0872665 upper=1.3089969 effort=1.5 velocity=3.59
- joint F3-L-MCP1: limit lower=-0.52 upper=1.57 effort=5.5 velocity=6.15 -> lower=-0.6108652 upper=1.6580628 effort=5.5 velocity=6.15
- joint F3-L-MCP2: limit lower=-0.61 upper=0.61 effort=6.0 velocity=3.59 -> lower=-0.6981317 upper=0.6108652 effort=6.0 velocity=3.59
- joint F3-L-PIP: limit lower=0 upper=1.92 effort=3.0 velocity=5.65 -> lower=-0.0872665 upper=1.8325957 effort=3.0 velocity=5.65
- joint F3-R-DIP: limit lower=0 upper=1.22 effort=1.5 velocity=3.59 -> lower=-0.0872665 upper=1.3089969 effort=1.5 velocity=3.59
- joint F3-R-MCP1: limit lower=-0.52 upper=1.57 effort=5.5 velocity=6.15 -> lower=-0.6108652 upper=1.6580628 effort=5.5 velocity=6.15
- joint F3-R-MCP2: limit lower=-0.61 upper=0.61 effort=6.0 velocity=3.59 -> lower=-0.6981317 upper=0.6108652 effort=6.0 velocity=3.59
- joint F3-R-PIP: limit lower=0 upper=1.92 effort=3.0 velocity=5.65 -> lower=-0.0872665 upper=1.8325957 effort=3.0 velocity=5.65
- joint F4-L-DIP: limit lower=0 upper=1.22 effort=1.5 velocity=3.59 -> lower=-0.0872665 upper=1.3089969 effort=1.5 velocity=3.59
- joint F4-L-MCP1: limit lower=-0.52 upper=1.57 effort=5.5 velocity=6.15 -> lower=-0.6108652 upper=1.6580628 effort=5.5 velocity=6.15
- joint F4-L-MCP2: limit lower=-0.61 upper=0.61 effort=6.0 velocity=3.59 -> lower=-0.6981317 upper=0.5235988 effort=6.0 velocity=3.59; origin xyz=0.0059875 0.078019 0.00395 rpy=3.1416 0 3.1416 -> xyz=0.0059875 0.078019 0.00395 rpy=3.1416 0 3.4034
- joint F4-L-PIP: limit lower=0 upper=1.92 effort=3.0 velocity=5.65 -> lower=-0.0872665 upper=1.8325957 effort=3.0 velocity=5.65
- joint F4-R-DIP: limit lower=0 upper=1.22 effort=1.5 velocity=3.59 -> lower=-0.0872665 upper=1.3089969 effort=1.5 velocity=3.59
- joint F4-R-MCP1: limit lower=-0.52 upper=1.57 effort=5.5 velocity=6.15 -> lower=-0.6108652 upper=1.6580628 effort=5.5 velocity=6.15
- joint F4-R-MCP2: limit lower=-0.61 upper=0.61 effort=6.0 velocity=3.59 -> lower=-0.6981317 upper=0.5235988 effort=6.0 velocity=3.59; origin xyz=0.008399 0.0778613 0.0023 rpy=0 0 0 -> xyz=0.008399 0.0778613 0.0023 rpy=0 0 0.2618
- joint F4-R-PIP: limit lower=0 upper=1.92 effort=3.0 velocity=5.65 -> lower=-0.0872665 upper=1.8325957 effort=3.0 velocity=5.65
- joint F5-L-DIP: limit lower=0 upper=1.22 effort=1.5 velocity=3.59 -> lower=-0.0872665 upper=1.3089969 effort=1.5 velocity=3.59
- joint F5-L-MCP1: limit lower=-0.52 upper=1.57 effort=5.5 velocity=6.15 -> lower=-0.6108652 upper=1.6580628 effort=5.5 velocity=6.15
- joint F5-L-MCP2: limit lower=-0.61 upper=0.61 effort=6.0 velocity=3.59 -> lower=-0.6981317 upper=0.6981317 effort=6.0 velocity=3.59; origin xyz=-0.01361 0.063366 0.00395 rpy=3.1416 0 3.1416 -> xyz=-0.01361 0.063366 0.00395 rpy=3.1416 0 3.7350
- joint F5-L-PIP: limit lower=0 upper=1.92 effort=3.0 velocity=5.65 -> lower=-0.0872665 upper=1.8325957 effort=3.0 velocity=5.65
- joint F5-R-DIP: limit lower=0 upper=1.22 effort=1.5 velocity=3.59 -> lower=-0.0872665 upper=1.3089969 effort=1.5 velocity=3.59
- joint F5-R-MCP1: limit lower=-0.52 upper=1.57 effort=5.5 velocity=6.15 -> lower=-0.6108652 upper=1.6580628 effort=5.5 velocity=6.15
- joint F5-R-MCP2: limit lower=-0.61 upper=0.61 effort=6.0 velocity=3.59 -> lower=-0.6981317 upper=0.6981317 effort=6.0 velocity=3.59; origin xyz=-0.0111988 0.0632092 0.0023 rpy=0 0 0 -> xyz=-0.0111988 0.0632092 0.0023 rpy=0 0 0.5934
- joint F5-R-PIP: limit lower=0 upper=1.92 effort=3.0 velocity=5.65 -> lower=-0.0872665 upper=1.8325957 effort=3.0 velocity=5.65
- joint PALM-L: limit lower=-1.22 upper=1.22 effort=10.0 velocity=2.5 -> lower=-0.7853982 upper=0.7853982 effort=10.0 velocity=2.5
- joint PALM-R: limit lower=-1.22 upper=1.22 effort=10.0 velocity=2.5 -> lower=-0.7853982 upper=0.7853982 effort=10.0 velocity=2.5
- joint WRIST-PALM-L: limit lower=-0.785 upper=0.785 effort=12.0 velocity=2.0 -> lower=-1.2217305 upper=1.2217305 effort=12.0 velocity=2.0
- joint WRIST-PALM-R: limit lower=-0.785 upper=0.785 effort=12.0 velocity=2.0 -> lower=-1.2217305 upper=1.2217305 effort=12.0 velocity=2.0

Commit message: fix: sync standalone hand housing inertia

File: Hand/Hand_left/URDF_L.urdf (robot description, URDF)
Before this commit: robot URDF_0605_L, 24 links, 23 joints
Links:
- link HOUSING-L: mass 0.5561357 -> 1.8

File: Hand/Hand_right/URDF_R.urdf (robot description, URDF)
Before this commit: robot URDF_0605_R, 24 links, 23 joints
Links:
- link HOUSING-R: mass 0.5561357 -> 1.8
