Commit message: fix: sync robot mass and inertia models

File: bimanualHand/openarm_hand_bimanual.urdf (robot description, URDF)
Before this commit: robot openarm_hand_bimanual, 62 links, 61 joints
Links:
- link HOUSING-L: mass 0.5561357 -> 1.8
- link HOUSING-R: mass 0.5561357 -> 1.8
- link openarm_left_base_link: mass 0.487784887988258 -> 1.14323
- link openarm_left_link1: mass 0.561428544234246 -> 1.14167
- link openarm_left_link2: mass 0.295592749115978 -> 0.277509
- link openarm_left_link3: mass 0.850916861288263 -> 1.07386
- link openarm_left_link4: mass 0.590845933035621 -> 0.634853
- link openarm_left_link5: mass 0.5803968030561 -> 0.05
- link openarm_right_base_link: mass 0.487784887988258 -> 1.14323
- link openarm_right_link1: mass 0.561428544234246 -> 1.14167
- link openarm_right_link2: mass 0.295592749115978 -> 0.277509
- link openarm_right_link3: mass 0.850916861288263 -> 1.07386
- link openarm_right_link4: mass 0.590845933035621 -> 0.634853
- link openarm_right_link5: mass 0.5803968030561 -> 0.05

Commit message: fix: align DM4340P motors and measured flange inertia

File: bimanualHand/openarm_hand_bimanual.urdf (robot description, URDF)
Before this commit: robot openarm_hand_bimanual, 62 links, 61 joints
Links:
- link openarm_left_link3: mass 1.07386 -> 1.09286
- link openarm_left_link4: mass 0.634853 -> 0.715853
- link openarm_left_link5: mass 0.05 -> 0.0445
- link openarm_right_link3: mass 1.07386 -> 1.09286
- link openarm_right_link4: mass 0.634853 -> 0.715853
- link openarm_right_link5: mass 0.05 -> 0.0445
Joints:
- joint openarm_left_joint3: limit lower=-1.5708 upper=1.5708 effort=27 velocity=5.4454 -> lower=-1.5708 upper=1.5708 effort=27 velocity=10.471975511966
- joint openarm_left_joint4: limit lower=0 upper=2.4435 effort=27 velocity=5.4454 -> lower=0 upper=2.4435 effort=27 velocity=10.471975511966
- joint openarm_left_joint5: limit lower=-1.5708 upper=1.5708 effort=7 velocity=20.944 -> lower=-1.5708 upper=1.5708 effort=27 velocity=10.471975511966
- joint openarm_right_joint3: limit lower=-1.5708 upper=1.5708 effort=27 velocity=5.4454 -> lower=-1.5708 upper=1.5708 effort=27 velocity=10.471975511966
- joint openarm_right_joint4: limit lower=0 upper=2.4435 effort=27 velocity=5.4454 -> lower=0 upper=2.4435 effort=27 velocity=10.471975511966
- joint openarm_right_joint5: limit lower=-1.5708 upper=1.5708 effort=7 velocity=20.944 -> lower=-1.5708 upper=1.5708 effort=27 velocity=10.471975511966
